Commit message: lidar and camera

File: rover_20_description/urdf/altyurur_20.urdf.xacro (robot description, xacro)
@@ -5,4 +5,7 @@
 <robot
   name="altyurur_20" xmlns:xacro="http://www.ros.org/wiki/xacro">
+  <xacro:include filename="$(find rover_20_description)/urdf/vlp16.urdf.xacro"/>
+  <xacro:property name="cameraSize" value="0.05"/>
+  <xacro:property name="cameraMass" value="0.1"/>
   <link
     name="base_link">
@@ -256,4 +259,37 @@
     <axis
       xyz="0 0 -1" />
+  </joint>
+  <vlp16 prefix="base" topic="/velodyne_points" hz="10" samples="440" gpu="false"/>
+  <joint name="base_laser_joint" type="fixed">
+    <origin xyz="0.325 -0.775 -0.035" rpy="0 0 0" />
+    <parent link="base_link"/>
+    <child link="base_laser_mount"/>
+  </joint>
+  <link name="camera">
+    <collision>
+      <origin xyz="0 0 0" rpy="0 0 0"/>
+      <geometry>
+        <box size="${cameraSize} ${cameraSize} ${cameraSize}"/>
+      </geometry>
+    </collision>
+    <visual>
+      <origin xyz="0 0 0" rpy="0 0 0"/>
+      <geometry>
+        <box size="${cameraSize} ${cameraSize} ${cameraSize}"/>
+      </geometry>
+      <material name="green"/>
+    </visual>
+    <inertial>
+      <mass value="${cameraMass}" />
+      <origin xyz="0 0 0" rpy="0 0 0"/>
+      <box_inertia m="${cameraMass}" x="${cameraSize}" y="${cameraSize}" z="${cameraSize}" />
+      <inertia ixx="1e-6" ixy="0" ixz="0" iyy="1e-6" iyz="0" izz="1e-6" />
+    </inertial>
+  </link>
+  <joint name="camera_joint" type="fixed">
+    <axis xyz="1 1 0" />
+    <origin xyz="0.325 -0.775 0.105" rpy="0 0 0"/>
+    <parent link="base_link"/>
+    <child link="camera"/>
   </joint>
   <transmission name="left_front_trans" type="SimpleTransmission">
@@ -326,3 +362,39 @@
     </plugin>
   </gazebo>
+  <gazebo reference="camera">
+     <sensor type="camera" name="camera">
+       <update_rate>30.0</update_rate>
+       <camera name="camera">
+         <horizontal_fov>1.3962634</horizontal_fov>
+         <image>
+           <width>800</width>
+           <height>800</height>
+           <format>R8G8B8</format>
+         </image>
+         <clip>
+           <near>0.02</near>
+           <far>300</far>
+         </clip>
+         <noise>
+           <type>gaussian</type>
+           <mean>0.0</mean>
+           <stddev>0.007</stddev>
+         </noise>
+       </camera>
+       <plugin name="camera_controller" filename="libgazebo_ros_camera.so">
+         <alwaysOn>true</alwaysOn>
+         <updateRate>0.0</updateRate>
+         <cameraName>/mybot/camera</cameraName>
+         <imageTopicName>camera_view</imageTopicName>
+         <cameraInfoTopicName>camera_info</cameraInfoTopicName>
+         <frameName>camera</frameName>
+         <hackBaseline>0.07</hackBaseline>
+         <distortionK1>0.0</distortionK1>
+         <distortionK2>0.0</distortionK2>
+         <distortionK3>0.0</distortionK3>
+         <distortionT1>0.0</distortionT1>
+         <distortionT2>0.0</distortionT2>
+       </plugin>
+     </sensor>
+   </gazebo>
 </robot>

Commit message: joint position finder codes added

File: rover_20_description/urdf/altyurur_20.urdf.xacro (robot description, xacro)
@@ -5,4 +5,7 @@
 <robot
   name="altyurur_20" xmlns:xacro="http://www.ros.org/wiki/xacro">
+  <xacro:include filename="$(find rover_20_description)/urdf/vlp16.urdf.xacro"/>
+  <xacro:property name="cameraSize" value="0.05"/>
+  <xacro:property name="cameraMass" value="0.1"/>
   <link
     name="base_link">
@@ -256,4 +259,37 @@
     <axis
       xyz="0 0 -1" />
+  </joint>
+  <vlp16 prefix="base" topic="/velodyne_points" hz="10" samples="440" gpu="false"/>
+  <joint name="base_laser_joint" type="fixed">
+    <origin xyz="0.325 -0.775 -0.035" rpy="0 0 0" />
+    <parent link="base_link"/>
+    <child link="base_laser_mount"/>
+  </joint>
+  <link name="camera">
+    <collision>
+      <origin xyz="0 0 0" rpy="0 0 0"/>
+      <geometry>
+        <box size="${cameraSize} ${cameraSize} ${cameraSize}"/>
+      </geometry>
+    </collision>
+    <visual>
+      <origin xyz="0 0 0" rpy="0 0 0"/>
+      <geometry>
+        <box size="${cameraSize} ${cameraSize} ${cameraSize}"/>
+      </geometry>
+      <material name="green"/>
+    </visual>
+    <inertial>
+      <mass value="${cameraMass}" />
+      <origin xyz="0 0 0" rpy="0 0 0"/>
+      <box_inertia m="${cameraMass}" x="${cameraSize}" y="${cameraSize}" z="${cameraSize}" />
+      <inertia ixx="1e-6" ixy="0" ixz="0" iyy="1e-6" iyz="0" izz="1e-6" />
+    </inertial>
+  </link>
+  <joint name="camera_joint" type="fixed">
+    <axis xyz="1 1 0" />
+    <origin xyz="0.325 -0.775 0.105" rpy="0 0 0"/>
+    <parent link="base_link"/>
+    <child link="camera"/>
   </joint>
   <transmission name="left_front_trans" type="SimpleTransmission">
@@ -301,5 +337,5 @@
    <gazebo>
     <plugin name="imu_controller" filename="libhector_gazebo_ros_imu.so">
-      <updateRate>50.0</updateRate>
+      <updateRate>30.0</updateRate>
       <bodyName>base_link</bodyName>
       <topicName>/imu/data</topicName>
@@ -314,5 +350,5 @@
   <gazebo>
     <plugin name="gps_controller" filename="libhector_gazebo_ros_gps.so">
-      <updateRate>40</updateRate>
+      <updateRate>30</updateRate>
       <bodyName>base_link</bodyName>
       <frameId>base_link</frameId>
@@ -326,3 +362,39 @@
     </plugin>
   </gazebo>
+  <gazebo reference="camera">
+     <sensor type="camera" name="camera">
+       <update_rate>30.0</update_rate>
+       <camera name="camera">
+         <horizontal_fov>1.3962634</horizontal_fov>
+         <image>
+           <width>800</width>
+           <height>800</height>
+           <format>R8G8B8</format>
+         </image>
+         <clip>
+           <near>0.02</near>
+           <far>300</far>
+         </clip>
+         <noise>
+           <type>gaussian</type>
+           <mean>0.0</mean>
+           <stddev>0.007</stddev>
+         </noise>
+       </camera>
+       <plugin name="camera_controller" filename="libgazebo_ros_camera.so">
+         <alwaysOn>true</alwaysOn>
+         <updateRate>0.0</updateRate>
+         <cameraName>/rover_20/camera</cameraName>
+         <imageTopicName>camera_view</imageTopicName>
+         <cameraInfoTopicName>camera_info</cameraInfoTopicName>
+         <frameName>camera</frameName>
+         <hackBaseline>0.07</hackBaseline>
+         <distortionK1>0.0</distortionK1>
+         <distortionK2>0.0</distortionK2>
+         <distortionK3>0.0</distortionK3>
+         <distortionT1>0.0</distortionT1>
+         <distortionT2>0.0</distortionT2>
+       </plugin>
+     </sensor>
+   </gazebo>
 </robot>

Commit message: Update altyurur_20.urdf.xacro

File: rover_20_description/urdf/altyurur_20.urdf.xacro (robot description, xacro)
@@ -260,9 +260,9 @@
       xyz="0 0 -1" />
   </joint>
-  <vlp16 prefix="base" topic="/velodyne_points" hz="10" samples="440" gpu="false"/>
+  <vlp16 prefix="base" topic="/velodyne_points" hz="10" samples="440" gpu="false" max_range="5.0" min_range="0.1" min_angle="-2.39982772" max_angle="2.39982772"/>
   <joint name="base_laser_joint" type="fixed">
-    <origin xyz="0.325 -0.775 -0.035" rpy="0 0 0" />
+    <origin xyz="0.325 -0.775 -0.035" rpy="0 0 0" /><!-- 0.325 -0.775 -0.035-->
     <parent link="base_link"/>
-    <child link="base_laser_mount"/>
+    <child link="velodyne"/>
   </joint>
   <link name="camera">
